File: 373brd.brd (EAGLE design)
At the start: 160 x 100 mm, 46 parts, among them U3 XC6210

Commit message: finished routing
Parts:
- removed JP1: (no value), pinhead:1X08
- removed JP3: (no value), pinhead:1X10
- removed LED5: Red, SparkFun-LED:LED-0603
- removed LED6, LED7, LED8: Green, SparkFun-LED:LED-0603
- removed POWER_HEAD: (no value), con-lstb:MA06-2
- removed R17, R18: (no value), resistor:R0603
- removed R4, R5, R6, R7: 1k, SparkFun-Resistors:0603-RES
- added ADC_HEAD1, ADC_HEAD2: (no value), pinhead:1X04
- added ADC_POWHEAD: (no value), pinhead:1X08
- added MPU_OUT: (no value), pinhead:1X10
- added U$2, U$4, U$6: APA102, SAUVE:APA102
- moved C18 75.1 mm to (29.0, 15.7), turned to 180 degrees
- moved R11 73.9 mm to (13.2, 11.9), turned to 90 degrees
- moved C17 68.9 mm to (28.7, 21.6)
- moved C8 61.1 mm to (22.4, 29.2)
- moved LED4 57.6 mm to (13.2, 8.38), turned to 180 degrees
- moved C1 51.4 mm to (17.8, 27.9), turned to 180 degrees
- moved C14 50.3 mm to (18.0, 34.3), turned to 180 degrees
- moved C13 47.0 mm to (18.0, 32.3), turned to 180 degrees
- moved C12 43.1 mm to (18.0, 30.0)
- moved BLE_OUT 41.8 mm to (18.8, 3.05), turned to 180 degrees
- moved R1 41.2 mm to (40.1, 3.30), turned to 270 degrees
- moved U$5 35.6 mm to (39.4, 12.7), turned to 180 degrees
- moved R8 34.9 mm to (3.81, 23.6), turned to 0 degrees
- moved R13 34.1 mm to (3.81, 33.3)
- moved R2 32.5 mm to (32.5, 3.30), turned to 270 degrees
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Connections:
- removed net +5V: POWER_HEAD.1, POWER_HEAD.10, POWER_HEAD.11, POWER_HEAD.12, POWER_HEAD.2, POWER_HEAD.3, POWER_HEAD.4, POWER_HEAD.5, POWER_HEAD.6, POWER_HEAD.7, POWER_HEAD.8, POWER_HEAD.9
- removed net 3.3V: R11.2, R4.1, R5.1
- removed net DIN: LED6.C
- removed net DIO5: R7.2
- removed net DOUT: LED5.C
- removed net N$139: LED8.A, R7.1
- removed net N$7: LED5.A, R4.2
- removed net N$8: LED6.A, R5.2
- removed net N$9: LED7.A, R6.1
- removed net PA0/U0RX: U$3.17
- removed net PA1/U0TX: U$3.18
- removed net RSSI: R6.2
- new net N$1: U$2.SDO, U$4.SDI
- new net N$2: U$2.CKO, U$4.CKI
- new net N$3: U$4.SDO, U$6.SDI
- new net N$4: U$4.CKO, U$6.CKI
- net +3V3: now also ADC_POWHEAD.1, ADC_POWHEAD.2, ADC_POWHEAD.3, ADC_POWHEAD.4, ADC_POWHEAD.5, ADC_POWHEAD.6, ADC_POWHEAD.7, ADC_POWHEAD.8, MPU_OUT.10, R11.2, U$2.VCC, U$4.VCC, U$6.VCC; no longer JP3.10
- net ADC0: now also ADC_HEAD1.4; no longer JP1.8
- net ADC1: now also ADC_HEAD1.3; no longer JP1.7
- net ADC2: now also ADC_HEAD1.2; no longer JP1.6
- net ADC3: now also ADC_HEAD1.1; no longer JP1.5
- net ADC4: now also ADC_HEAD2.4; no longer JP1.4
- net ADC5: now also ADC_HEAD2.3; no longer JP1.3
- net ADC6: now also ADC_HEAD2.2; no longer JP1.2
- net ADC7: now also ADC_HEAD2.1; no longer JP1.1
- net ADC8: no longer R17.2
- net ADC9: no longer R18.2
- net BLE_UART_RX: now also U$3.17
- net BLE_UART_TX: now also U$3.18
- net GND: now also MPU_OUT.1, MPU_OUT.2, MPU_OUT.4, MPU_OUT.9, U$2.GND, U$4.GND, U$6.GND; no longer JP3.1, JP3.2, JP3.4, JP3.9, LED7.C, LED8.C, R17.1, R18.1
- net I2C_CLK_MPU: now also MPU_OUT.8; no longer JP3.8
- net I2C_DATA_MPU: now also MPU_OUT.7; no longer JP3.7
- net MPU_INT: now also MPU_OUT.3; no longer JP3.3
- net SPI0_CLK: now also U$2.CKI
- net SPI_0_TX: now also U$2.SDI
Routing:
- net +3V3: track 56.3 -> 171.4 mm, vias 2 -> 4
- net GND: track 39.9 -> 98.6 mm, vias 1 -> 4
- net PC0/TCK/SWCLK: track 0.00 -> 38.6 mm, vias 0 -> 3
- net +5V: track 27.9 -> 0.00 mm
- net SPI_0_TX: track 0.00 -> 24.0 mm, vias 0 -> 2
- net SPI0_CLK: track 0.00 -> 23.3 mm, vias 0 -> 2
- net T_OSC1: track 28.1 -> 5.33 mm, vias 2 -> 0
- net T_VDDC: track 0.00 -> 22.4 mm
- net T_OSC0: track 26.5 -> 7.09 mm
- net MPU_INT: track 20.7 -> 38.4 mm
- net ADC4: track 0.00 -> 16.9 mm
- net ADC5: track 0.00 -> 16.0 mm
- net I2C_CLK_MPU: track 40.0 -> 24.8 mm, vias 0 -> 2
- net I2C_DATA_MPU: track 38.0 -> 23.6 mm, vias 2 -> 0
- net BLE_UART_TX: track 0.00 -> 13.9 mm
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- removed copper zone on layer 16, net +3V3

Commit message: done for real
Parts:
- moved LED4 1.02 mm to (13.2, 7.37)
- moved R11 1.02 mm to (13.2, 10.9)
- moved C18 0.41 mm to (28.5, 15.7)
- moved R12 0.14 mm to (3.71, 15.9)
Routing:
- net GND: track 98.6 -> 138.7 mm, vias 4 -> 10
- net +3V3: track 171.4 -> 184.7 mm, vias 4 -> 6
- net PC3/TDO/SWO: track 20.2 -> 25.2 mm, vias 2 -> 3
- net MPU_INT: track 38.4 -> 42.9 mm
- net RESET: track 22.4 -> 24.0 mm
- net PC1/TMS/SWDIO: track 38.7 -> 40.1 mm
- net BATT_IN: track 32.0 -> 31.1 mm, vias 2 -> 0
- net BLE_UART_TX: track 13.9 -> 13.2 mm
- net PC2/TDI: track 29.4 -> 30.1 mm, vias 4 -> 3
Other:
- board size 160 x 100 mm -> 50.4 x 39.6 mm
- board text added: "GloveBoard, rev0 Designed by James Connolly Laid out by James Connolly"

Commit message: new brd
Parts:
- removed BLE_OUT: (no value), pinhead:1X06
- removed LED4: Red, SparkFun-LED:LED-0603
- removed R11: 1k, SparkFun-Resistors:0603-RES
- added D1, D2: IR, SparkFun-LED:LED-1206
- added R5: (no value), resistor:R0603
- added RF_OUT: (no value), pinhead:2X04
Connections:
- removed net BLE_UART_RX: BLE_OUT.3, U$3.17
- removed net BLE_UART_TX: BLE_OUT.2, U$3.18
- removed net N$6: LED4.A, R11.1
- removed net PF0: U$3.28
- removed net PF1: U$3.29
- removed net PF2: U$3.30
- removed net PF3: U$3.31
- new net CE: RF_OUT.3, U$3.31
- new net CS: RF_OUT.4, U$3.17
- new net IRQ_RF: RF_OUT.8, U$3.18
- new net MISO_RF: RF_OUT.7, U$3.28
- new net MOSI_RF: RF_OUT.6, U$3.29
- new net N$5: D1.A, D2.C
- new net N$7: D2.A, R5.1
- new net SCK: RF_OUT.5, U$3.30
- net +3V3: now also R5.2, RF_OUT.2; no longer R11.2
- net BATT_IN: no longer BLE_OUT.4
- net GND: now also D1.C, RF_OUT.1; no longer BLE_OUT.1, BLE_OUT.5, BLE_OUT.6, LED4.C
Routing:
- net CS: track 0.00 -> 21.4 mm
- net MOSI_RF: track 0.00 -> 18.9 mm, vias 0 -> 1
- net BATT_IN: track 31.1 -> 14.2 mm
- net MISO_RF: track 0.00 -> 14.8 mm, vias 0 -> 2
- net +3V3: track 184.7 -> 198.7 mm, vias 6 -> 7
- net CE: track 0.00 -> 13.8 mm, vias 0 -> 1
- net SCK: track 0.00 -> 13.5 mm, vias 0 -> 1
- net BLE_UART_TX: track 13.2 -> 0.00 mm
- net BLE_UART_RX: track 12.4 -> 0.00 mm
- net IRQ_RF: track 0.00 -> 10.7 mm
- net N$5: track 0.00 -> 2.45 mm
- net N$7: track 0.00 -> 2.02 mm
- net N$6: track 1.83 -> 0.00 mm
- net MPU_INT: track 42.9 -> 44.1 mm
- net GND: track 138.7 -> 139.8 mm
