File: 373brd.sch (EAGLE design)
At the start: 46 parts, among them U3 XC6210

Commit message: finished routing
Parts:
- removed JP1: (no value), pinhead:PINHD-1X8
- removed LED5: Red, SparkFun-LED:LED-RED0603
- removed LED6, LED7, LED8: Green, SparkFun-LED:LED-GREEN0603
- removed POWER_HEAD: (no value), con-lstb:MA06-2
- removed R17, R18: (no value), resistor:R-US_R0603
- removed R4, R5, R6, R7: 1k, SparkFun-Resistors:1KOHM1/10W1%(0603)
- added ADC_HEAD1, ADC_HEAD2: (no value), pinhead:PINHD-1X4
- added ADC_POWHEAD: (no value), pinhead:PINHD-1X8
- added U$2, U$4, U$6: APA102, SAUVE:APA102
- renumbered JP3 to MPU_OUT
Connections:
- removed net +5V: POWER_HEAD.1, POWER_HEAD.10, POWER_HEAD.11, POWER_HEAD.12, POWER_HEAD.2, POWER_HEAD.3, POWER_HEAD.4, POWER_HEAD.5, POWER_HEAD.6, POWER_HEAD.7, POWER_HEAD.8, POWER_HEAD.9
- removed net 3.3V: R11.2, R4.1, R5.1
- removed net DIN: LED6.C
- removed net DIO5: R7.2
- removed net DOUT: LED5.C
- removed net N$139: LED8.A, R7.1
- removed net N$7: LED5.A, R4.2
- removed net N$8: LED6.A, R5.2
- removed net N$9: LED7.A, R6.1
- removed net PA0/U0RX: U$3.PA0/U0RX
- removed net PA1/U0TX: U$3.PA1/U0TX
- removed net RSSI: R6.2
- new net N$1: U$2.SDO, U$4.SDI
- new net N$2: U$2.CKO, U$4.CKI
- new net N$3: U$4.SDO, U$6.SDI
- new net N$4: U$4.CKO, U$6.CKI
- net +3V3: now also ADC_POWHEAD.1, ADC_POWHEAD.2, ADC_POWHEAD.3, ADC_POWHEAD.4, ADC_POWHEAD.5, ADC_POWHEAD.6, ADC_POWHEAD.7, ADC_POWHEAD.8, R11.2, U$2.VCC, U$4.VCC, U$6.VCC
- net ADC0: now also ADC_HEAD1.4; no longer JP1.8
- net ADC1: now also ADC_HEAD1.3; no longer JP1.7
- net ADC2: now also ADC_HEAD1.2; no longer JP1.6
- net ADC3: now also ADC_HEAD1.1; no longer JP1.5
- net ADC4: now also ADC_HEAD2.4; no longer JP1.4
- net ADC5: now also ADC_HEAD2.3; no longer JP1.3
- net ADC6: now also ADC_HEAD2.2; no longer JP1.2
- net ADC7: now also ADC_HEAD2.1; no longer JP1.1
- net ADC8: no longer R17.2
- net ADC9: no longer R18.2
- net BLE_UART_RX: now also U$3.PA0/U0RX
- net BLE_UART_TX: now also U$3.PA1/U0TX
- net GND: now also U$2.GND, U$4.GND, U$6.GND; no longer LED7.C, LED8.C, R17.1, R18.1
- net SPI0_CLK: now also U$2.CKI
- net SPI_0_TX: now also U$2.SDI
Other:
- moved on the sheet: C8, C9

Commit message: new brd
Parts:
- removed BLE_OUT: (no value), pinhead:PINHD-1X6
- removed LED4: Red, SparkFun-LED:LED-RED0603
- removed R11: 1k, SparkFun-Resistors:1KOHM1/10W1%(0603)
- added D1, D2: IR, SparkFun-LED:LED-BLUE1206
- added R5: (no value), resistor:R-US_R0603
- added RF_OUT: (no value), pinhead:PINHD-2X4
Connections:
- removed net BLE_UART_RX: BLE_OUT.3, U$3.PA0/U0RX
- removed net BLE_UART_TX: BLE_OUT.2, U$3.PA1/U0TX
- removed net N$6: LED4.A, R11.1
- removed net PF0: U$3.PF0
- removed net PF1: U$3.PF1
- removed net PF2: U$3.PF2
- removed net PF3: U$3.PF3
- new net CE: RF_OUT.3, U$3.PF3
- new net CS: RF_OUT.4, U$3.PA0/U0RX
- new net IRQ_RF: RF_OUT.8, U$3.PA1/U0TX
- new net MISO_RF: RF_OUT.7, U$3.PF0
- new net MOSI_RF: RF_OUT.6, U$3.PF1
- new net N$5: D1.A, D2.C
- new net N$7: D2.A, R5.1
- new net SCK: RF_OUT.5, U$3.PF2
- net +3V3: now also R5.2, RF_OUT.2; no longer R11.2
- net BATT_IN: no longer BLE_OUT.4
- net GND: now also D1.C, RF_OUT.1; no longer BLE_OUT.1, BLE_OUT.5, BLE_OUT.6, LED4.C
